Commit message: 2d.urdf

File: src/taobot_link/move_base_config/2d.urdf (robot description, URDF)
Before this commit: robot cartographer_backpack_2d, 2 links, 1 joints
Joints:
- joint horizontal_laser_link_joint: child horizontal_laser_link -> laser; parent laser -> base_link

Commit message: 2d.urdf

File: src/taobot_link/move_base_config/2d.urdf (robot description, URDF)
Before this commit: robot cartographer_backpack_2d, 3 links, 1 joints
Links:
- removed link horizontal_laser_link
- link base_link: geometry visual cylinder length=0.05 radius=0.03

Commit message: modified to add head camera

File: src/taobot_link/move_base_config/2d.urdf (robot description, URDF)
Before this commit: robot cartographer_backpack_2d, 2 links, 1 joints
Joints:
- added joint horizontal_camera_link_joint: type fixed, parent base_link, child head_camera, origin xyz=0.1007 0.2 0.0558

Commit message: head_camera didnt add correctly

File: src/taobot_link/move_base_config/2d.urdf (robot description, URDF)
Before this commit: robot cartographer_backpack_2d, 2 links, 2 joints
Links:
- added link head_camera
